File: pcb/battEliminator.kicad_pcb (KiCad board)
At the start: 2 copper layers, 31 x 58 mm, 28 parts, among them J1 PWR, J2 +, J3 GND, U1 AP63200WU

Commit message: Fixed size and position of the radio battery pads
Parts:
- moved J2 4.00 mm to (119.2, 134.0)
- moved J3 4.00 mm to (136.2, 134.0)
Routing:
- net Net-(D3-K): track 31.7 -> 25.5 mm
- net GND: vias 167 -> 158
Other:
- board text added: "Battery Eliminator for NavComm NC-55A www.deadbadger.cz Kajus v0.2 2024"
- board text removed: "Battery Eliminator for NavComm NC-55A www.deadbadger.cz Kajus v0.1 2024"
